File: kicad/compander.sch (KiCad schematic (older format))
At the start: 49 parts, among them P101 CONN_6, P102 CONN_6, U101 SA571

Commit message: mod: Schematics
Parts:
- removed P101, P102: CONN_6, symbol CONN_6
